Commit message: Added STLs, updated gitignore, added sym_jacob

File: open_manipulator_x.urdf (robot description, URDF)
Before this commit: robot open_manipulator_x, 9 links, 8 joints
Links:
- link gripper_left_link: geometry collision mesh filename=meshes/open_manipulator_x/gripper_left_palm.stl scale=0.001 0.001 0.001; visual mesh filename=meshes/open_manipulator_x/gripper_left_palm.stl scale=0.001 0.001 0.001
- link gripper_right_link: geometry collision mesh filename=meshes/open_manipulator_x/gripper_right_palm.stl scale=0.001 0.001 0.001; visual mesh filename=meshes/open_manipulator_x/gripper_right_palm.stl scale=0.001 0.001 0.001
- link link1: geometry collision mesh filename=meshes/open_manipulator_x/link1.stl scale=0.001 0.001 0.001; visual mesh filename=meshes/open_manipulator_x/link1.stl scale=0.001 0.001 0.001
- link link2: geometry collision mesh filename=meshes/open_manipulator_x/link2.stl scale=0.001 0.001 0.001; visual mesh filename=meshes/open_manipulator_x/link2.stl scale=0.001 0.001 0.001
- link link3: geometry collision mesh filename=meshes/open_manipulator_x/link3.stl scale=0.001 0.001 0.001; visual mesh filename=meshes/open_manipulator_x/link3.stl scale=0.001 0.001 0.001
- link link4: geometry collision mesh filename=meshes/open_manipulator_x/link4.stl scale=0.001 0.001 0.001; visual mesh filename=meshes/open_manipulator_x/link4.stl scale=0.001 0.001 0.001
- link link5: geometry collision mesh filename=meshes/open_manipulator_x/link5.stl scale=0.001 0.001 0.001; visual mesh filename=meshes/open_manipulator_x/link5.stl scale=0.001 0.001 0.001
